Commit message: add new simulation env.

File: simpledog/urdf/quadruped_model.urdf.xacro (robot description, xacro)
@@ -43,19 +43,20 @@
   <!-- <xacro:arg name="camera_visual" default="false"/> -->
   <!-- <xacro:arg name="imu_visual"    default="false"/> -->
-  <!-- <xacro:arg name="kinect_enabled"    default="true"/> -->
+  <xacro:arg name="kinect_enabled"    default="true"/>
     <xacro:include filename="$(find simpledog)/urdf/simpledog_gazebo.urdf.xacro" />
     <xacro:include filename="$(find simpledog)/urdf/joint_gazebo.urdf.xacro" />
-    <!-- <xacro:include filename="$(find simpledog)/urdf/kinect.urdf.xacro"/> -->
+    <xacro:include filename="$(find simpledog)/urdf/kinect.urdf.xacro"/>
     <xacro:include filename="$(find simpledog)/urdf/foot_sensor_gazebo.urdf.xacro" />
     <!--load kinect urdf-->
-    <!-- <xacro:if value="$(arg kinect_enabled)">
+    <xacro:if value="$(arg kinect_enabled)">
       <xacro:kinect_camera prefix="camera" robot_namespace="$(arg robot_namespace)"/>
       <joint name="kinect_frame_joint" type="fixed">
-        <origin xyz="0.5 0 0.075" rpy="0 0.8 0" />
+        <origin xyz="0.5 0 0.075" rpy="0 0.6 0" /> // 30 degree
         <parent link="base_link"/>
         <child link="camera_link"/>
       </joint>
-    </xacro:if> -->
-  <link name="zed_base_link">
+    </xacro:if>
+<!--load real zed camera urdf-->
+  <!-- <link name="zed_base_link">
     <origin xyz="0 0 0" rpy="0 0 0"/>
   </link>
@@ -64,5 +65,5 @@
     <parent link="base_link"/>
     <child link="zed_base_link"/>
-  </joint>
+  </joint> -->
   <!-- simple dog joints macros configure the joint driver and param-->
   <xacro:simpledog_joint joint_prefix="front_left_1_"> </xacro:simpledog_joint>
